File: parvus_amp/parvus_amp.sch (KiCad schematic (older format))
At the start: 43 parts, among them J1 input, J2 output, J3 powersupply, U1 LM3886

Commit message: Transition to TDA7293
Parts:
- removed C1, C8: 15p, Capacitor_THT:C_Disc_D3.8mm_W2.6mm_P2.50mm, symbol Device:C
- removed C10, C13: 2m2, Capacitor_THT:CP_Radial_D16.0mm_P7.50mm, symbol Device:CP1
- removed C11, C14, C3: 100n, Capacitor_THT:C_Rect_L7.0mm_W3.5mm_P5.00mm, symbol Device:C
- removed C12, C15, C9: 100u, Capacitor_THT:CP_Radial_D8.0mm_P3.50mm, symbol Device:CP1
- removed C2: 220n, Capacitor_THT:C_Rect_L7.0mm_W3.5mm_P5.00mm, symbol Device:C
- removed C4, C7: 470u, Capacitor_THT:CP_Radial_D8.0mm_P3.50mm, symbol Device:CP1
- removed C5: 220p, Capacitor_THT:C_Disc_D4.3mm_W1.9mm_P5.00mm, symbol Device:C
- removed C6: 1n, Capacitor_THT:C_Disc_D4.3mm_W1.9mm_P5.00mm, symbol Device:C
- removed D1, D2: 1N5404, Diode_THT:D_DO-201AD_P12.70mm_Horizontal, symbol Diode:1N5404
- removed D3: BZX85C16, Diode_THT:D_DO-35_SOD27_P7.62mm_Horizontal, symbol Device:D_Zener
- removed J1: input, TerminalBlock_Phoenix:TerminalBlock_Phoenix_PT-1,5-3-3.5-H_1x03_P3.50mm_Horizontal, symbol Connector_Generic:Conn_01x03
- removed J2: output, Connector_Phoenix_MC:PhoenixContact_MCV_1,5_2-G-3.5_1x02_P3.50mm_Vertical, symbol Connector:Screw_Terminal_01x02
- removed J3: powersupply, Connector_Phoenix_MC:PhoenixContact_MCV_1,5_3-G-3.5_1x03_P3.50mm_Vertical, symbol Connector:Screw_Terminal_01x03
- removed L1: 2u, Inductor_THT:L_Axial_L12.0mm_D5.0mm_P15.24mm_Horizontal_Fastron_MISC, symbol Device:L
- removed R1, R13: 1k6, Resistor_THT:R_Axial_DIN0207_L6.3mm_D2.5mm_P7.62mm_Horizontal, symbol Device:R
- removed R10, R6: 499, Resistor_THT:R_Axial_DIN0207_L6.3mm_D2.5mm_P10.16mm_Horizontal, symbol Device:R
- removed R11, R7: 7k5, Resistor_THT:R_Axial_DIN0207_L6.3mm_D2.5mm_P10.16mm_Horizontal, symbol Device:R
- removed R12, R3: 10, Resistor_THT:R_Axial_DIN0207_L6.3mm_D2.5mm_P10.16mm_Horizontal, symbol Device:R
- removed R14: 7k5, Resistor_THT:R_Axial_DIN0207_L6.3mm_D2.5mm_P7.62mm_Horizontal, symbol Device:R
- removed R2, R9: 4.7, Resistor_THT:R_Axial_DIN0411_L9.9mm_D3.6mm_P15.24mm_Horizontal, symbol Device:R
- removed R4, R5: 100, Resistor_THT:R_Axial_DIN0207_L6.3mm_D2.5mm_P7.62mm_Horizontal, symbol Device:R
- removed R8: 100k, Resistor_THT:R_Axial_DIN0207_L6.3mm_D2.5mm_P7.62mm_Horizontal, symbol Device:R
- removed U1: LM3886, Package_TO_SOT_THT:TO-220-11_P3.4x5.08mm_StaggerOdd_Lead4.85mm_Vertical, symbol Amplifier_Audio:LM3886
- added C?: 3p3, Capacitor_THT:C_Disc_D3.8mm_W2.6mm_P2.50mm, symbol Device:C
- added C? (x5): 100n, Capacitor_THT:C_Rect_L4.6mm_W3.0mm_P2.50mm_MKS02_FKP02, symbol Device:C
- added C?: 100n, Capacitor_THT:C_Disc_D5.1mm_W3.2mm_P5.00mm, symbol Device:C
- added C? (x3): 10u, Capacitor_THT:CP_Radial_D5.0mm_P2.00mm, symbol Device:CP
- added C?: 220p, Capacitor_THT:C_Disc_D3.8mm_W2.6mm_P2.50mm, symbol Device:C
- added C? (x3): 47u, Capacitor_THT:CP_Radial_D6.3mm_P2.50mm, symbol Device:CP
- added C? (x2): 100u, Capacitor_THT:CP_Radial_D10.0mm_P5.00mm, symbol Device:CP
- added C? (x2): 2m2, Capacitor_THT:CP_Radial_D10.0mm_P5.00mm, symbol Device:CP
- added C?: 220u, Capacitor_THT:CP_Radial_D6.3mm_P2.50mm, symbol Device:CP
- added D? (x2): 1N5404, Diode_THT:D_DO-35_SOD27_P7.62mm_Horizontal, symbol Device:D
- added D?: 1N4148, symbol Device:D
- added J? (x2): Conn_01x03, symbol Connector_Generic:Conn_01x03
- added J?: Conn_01x02, symbol Connector_Generic:Conn_01x02
- added L?: 4u, Inductor_THT:L_Axial_L20.3mm_D12.7mm_P7.62mm_Vertical_Vishay_IHA-201, symbol Device:L
- added R? (x2): 3.9, Resistor_THT:R_Axial_DIN0207_L6.3mm_D2.5mm_P10.16mm_Horizontal, symbol Device:R
- added R?: 10k, Resistor_THT:R_Axial_DIN0204_L3.6mm_D1.6mm_P5.08mm_Horizontal, symbol Device:R
- added R? (x2): 12k, Resistor_THT:R_Axial_DIN0207_L6.3mm_D2.5mm_P10.16mm_Horizontal, symbol Device:R
- added R?: 20k, Resistor_THT:R_Axial_DIN0204_L3.6mm_D1.6mm_P5.08mm_Horizontal, symbol Device:R
- added R? (x2): 499, Resistor_THT:R_Axial_DIN0207_L6.3mm_D2.5mm_P10.16mm_Horizontal, symbol Device:R
- added R?: 10, Resistor_THT:R_Axial_DIN0207_L6.3mm_D2.5mm_P10.16mm_Horizontal, symbol Device:R
- added R?: 30k, Resistor_THT:R_Axial_DIN0204_L3.6mm_D1.6mm_P5.08mm_Horizontal, symbol Device:R
- added U?: TDA7293, Package_TO_SOT_THT:TO-220-15_P2.54x2.54mm_StaggerOdd_Lead4.58mm_Vertical, symbol tda7293:TDA7293
- renumbered LOGO2 to LOGO?, LOGO1 to LOGO?, MK1 to MK?, MK3 to MK?, MK4 to MK?, MK2 to MK?
Connections:
- net labels added: +pwvs, +vs, -pwvs, -vs, GNDD, in_l, ingnd_l, out_l, overload
- net labels removed: VCC, VEE
- wire segments 115 -> 124
- no-connect marks 0 -> 1
Other:
- note added: "1.32 HP"
- note added: "1.44 SHP"
- note added: "Place the capacitors as\nclose as possible to IC\npins"
- note added: "Return to supply bypass \ncapacitor ground"
- note removed: "Fz=1.6e6\nFp=6.6e6"

Commit message: WIP: Component placement.
Signed-off-by: Nenad Radulovic <nenad.b.radulovic@gmail.com>
Parts:
- removed C? (x2): 100n, Capacitor_THT:C_Rect_L4.6mm_W3.0mm_P2.50mm_MKS02_FKP02, symbol Device:C
- removed C?: 220p, Capacitor_THT:C_Disc_D3.8mm_W2.6mm_P2.50mm, symbol Device:C
- removed C? (x2): 47u, Capacitor_THT:CP_Radial_D6.3mm_P2.50mm, symbol Device:CP
- removed C? (x2): 100u, Capacitor_THT:CP_Radial_D10.0mm_P5.00mm, symbol Device:CP
- removed J?: Conn_01x02, symbol Connector_Generic:Conn_01x02
- added C5, C6: 22n, Capacitor_THT:C_Rect_L4.6mm_W3.0mm_P2.50mm_MKS02_FKP02, symbol Device:C
- added C9: 3p3, Capacitor_THT:C_Disc_D3.8mm_W2.6mm_P2.50mm, symbol Device:C
- added D4: BZX85C15, Diode_THT:D_DO-41_SOD81_P10.16mm_Horizontal, symbol Device:D_Zener
- added J1: input, Connector_Phoenix_MC:PhoenixContact_MCV_1,5_3-G-3.5_1x03_P3.50mm_Vertical, symbol Connector_Generic:Conn_01x03
- added J3: output, Connector_Phoenix_MC:PhoenixContact_MCV_1,5_2-G-3.81_1x02_P3.81mm_Vertical, symbol Connector_Generic:Conn_01x02
- added R1, R2: 499, Resistor_THT:R_Axial_DIN0207_L6.3mm_D2.5mm_P10.16mm_Horizontal, symbol Device:R
- added R13: 10k, Resistor_THT:R_Axial_DIN0204_L3.6mm_D1.6mm_P5.08mm_Horizontal, symbol Device:R
- C1, C2: renamed from C?; footprint Capacitor_THT:CP_Radial_D10.0mm_P5.00mm -> Capacitor_THT:CP_Radial_D16.0mm_P7.50mm
- C3, C4: renamed from C?; value 100n -> 220n
- D3: renamed from D?; footprint (none) -> Diode_THT:D_DO-35_SOD27_P7.62mm_Horizontal
- J2: renamed from J?; value Conn_01x03 -> power; footprint (none) -> Connector_Phoenix_MC:PhoenixContact_MCV_1,5_3-G-3.81_1x03_P3.81mm_Vertical
- J4: renamed from J?; value Conn_01x03 -> ctrl; footprint (none) -> Connector_PinHeader_2.54mm:PinHeader_1x04_P2.54mm_Vertical; symbol Connector_Generic:Conn_01x03 -> Connector_Generic:Conn_01x04
- R11: renamed from R?; value 30k -> 47k
- R12: renamed from R?; value 20k -> 30k
- R8: renamed from R?; value 10k -> 15k
- gave numbers to parts that had none: 25
Connections:
- net +vs is gone; now on net +pwvs: U1.7 (+Vs)
- net -vs is gone; now on net -pwvs: U1.8 (-Vs)
- net GNDPWR is gone; now on net GNDD: C1.2, C13.2, C15.2, C2.1, C3.2, C4.1, J2.2 (Pin_2)
- net +pwvs: now also C5.1
- net -pwvs: now also C6.2
- net GNDD: now also C5.2, C6.1, J1.3 (Pin_3), J3.2 (Pin_2), R13.1, R2.1
- net at U1.12 (bldr): no longer C11.2
- net preout: now reaches C10.2, D1.2 (A), D2.1 (K), L1.1, R6.2, R7.1, R9.2, U1.14
- net preout: now also C11.2
- net at R3.1, R5.1, U1.3 (+): now also C9.2
- net at D3.1 (K), R11.1, R12.1: now also D4.2 (A), R13.2; no longer J4.2 (Pin_2)
- net in_l renamed input
- net input: now also J1.1 (Pin_1), R1.2
- net ingnd_l renamed sgnd
- net sgnd: now also C9.1, J1.2 (Pin_2), R1.1, R2.2
- net out_l renamed out
- net out: now also J3.1 (Pin_1)
- net overload: no longer names the net of U1.5 (clip)
- net overload: now also J4.4 (Pin_4)
- new net: D4.1 (K), J4.2 (Pin_2)
- no-connect marks 1 -> 2
Other:
- moved on the sheet: C1, C10, C11, C12, C13, C14, C15, C2, C3, C4, C7, C8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

Commit message: WIP: Routing components
Parts:
- removed C4: 220n, Capacitor_THT:C_Rect_L4.6mm_W3.0mm_P2.50mm_MKS02_FKP02, symbol Device:C
- removed C6: 22n, Capacitor_THT:C_Rect_L4.6mm_W3.0mm_P2.50mm_MKS02_FKP02, symbol Device:C
- removed C9: 3p3, Capacitor_THT:C_Disc_D3.8mm_W2.6mm_P2.50mm, symbol Device:C
- removed D2: 1N5404, Diode_THT:D_DO-35_SOD27_P7.62mm_Horizontal, symbol Device:D
- removed R1, R2, R3: 499, Resistor_THT:R_Axial_DIN0207_L6.3mm_D2.5mm_P10.16mm_Horizontal, symbol Device:R
- added C15: 220n, Capacitor_THT:C_Rect_L4.6mm_W3.0mm_P2.50mm_MKS02_FKP02, symbol Device:C
- added C16: 22n, Capacitor_THT:C_Rect_L4.6mm_W3.0mm_P2.50mm_MKS02_FKP02, symbol Device:C
- added C5: 220p, Capacitor_THT:C_Disc_D3.8mm_W2.6mm_P2.50mm, symbol Device:C
- added D4: 1N5404, Diode_THT:D_DO-201AD_P12.70mm_Horizontal, symbol Device:D
- added R11: 10, Resistor_THT:R_Axial_DIN0207_L6.3mm_D2.5mm_P10.16mm_Horizontal, symbol Device:R
- added R6: 100, Resistor_THT:R_Axial_DIN0207_L6.3mm_D2.5mm_P10.16mm_Horizontal, symbol Device:R
- added R7: 12k, Resistor_THT:R_Axial_DIN0207_L6.3mm_D2.5mm_P10.16mm_Horizontal, symbol Device:R
- C1: renamed from C12; Manufacturer Multicomp:MCGPR16V106M5X11 -> Multicomp: MCGPR35V106M5X11; Supplier1 Farnell:9451056 -> Farnell: 9451242
- C10: renamed from C15; Manufacturer AVX:SR211C104KAR -> AVX: SR211C104KAR; Supplier1 Farnell:1006004 -> Farnell: 1100408
- C11: renamed from C1; Manufacturer Rybicon:35YXF220MEFC10X12.5 -> Rybicon: 50YXJ2200M16X35.5; Supplier1 Farnel:1144628 -> Farnel: 2346272; Voltage 35V -> 50V
- C12: renamed from C3; Manufacturer WIMA:MKS0C031000C00KSSD -> WIMA: MKS0C032200C00KSSD; Supplier1 Farnell:1006004 -> Farnell: 1890123
- C13: renamed from C5; Manufacturer WIMA:MKS0C031000C00KSSD -> WIMA: MKS0C022200B00KSSD; Supplier1 Farnell:1006004 -> Farnell: 1006001
- C14: value 10u -> 2m2; footprint Capacitor_THT:CP_Radial_D5.0mm_P2.00mm -> Capacitor_THT:CP_Radial_D16.0mm_P7.50mm; Manufacturer Multicomp:MCGPR16V106M5X11 -> Rybicon: 50YXJ2200M16X35.5; Supplier1 Farnell:9451056 -> Farnel: 2346272; Voltage 35V -> 50V
- C2: value 2m2 -> 10u; footprint Capacitor_THT:CP_Radial_D16.0mm_P7.50mm -> Capacitor_THT:CP_Radial_D5.0mm_P2.00mm; Manufacturer Rybicon:35YXF220MEFC10X12.5 -> Multicomp: MCGPR35V106M5X11; Supplier1 Farnel:1144628 -> Farnell: 9451242
- C4: renamed from C11; Manufacturer Rybicon:50YXF47MEFC6.3X11 -> Rybicon: 63YXJ47M6.3X11; Supplier1 Farnell:1144633 -> Farnell: 2346274; Voltage 50V -> 63V
- C6: renamed from C7; value 10u -> 3u3; Manufacturer Rybicon:50YXF10MEFC5X11 -> Rybicon: 50YXJ3R3M5X11; Supplier1 Farnell:1144632 -> Farnell: 2346267
- C7: renamed from C8; value 220u -> 470u; Manufacturer Rybicon:10YXF220MEFC6.3X11 -> Rybicon:10YXJ470M6.3X11; Supplier1 Farnel:1144609 -> Farnel: 2346252
- C8: renamed from C10; Manufacturer Kemet:C315C339D2G5TA -> Kemet: C315C339D2G5TA; Supplier1 Farnell:2819636 -> Farnell: 2819636
- C9: renamed from C13; Manufacturer WIMA:MKS0C031000C00KSSD -> WIMA: MKS0C031000C00KSSD; Supplier1 Farnell:1006004 -> Farnell: 1006004
- D1: renamed from D3; Manufacturer (none) -> ON Semiconductor: 1N4148TA; Supplier1 (none) -> Farnell: 2322485
- D2: renamed from D4; value BZX85C15 -> BZX79C15; footprint Diode_THT:D_DO-41_SOD81_P10.16mm_Horizontal -> Diode_THT:D_DO-35_SOD27_P7.62mm_Horizontal; Manufacturer (none) -> ON Semuconductor: BZX79C15; Supplier1 (none) -> Farnell: 1467595
- D3: renamed from D1; footprint Diode_THT:D_DO-35_SOD27_P7.62mm_Horizontal -> Diode_THT:D_DO-201AD_P12.70mm_Horizontal; Manufacturer (none) -> ON Semiconductor: 1N5404RL; Supplier1 (none) -> Farnell: 9556141
- J2: renamed from J1; Manufacturer (none) -> Phoenix: 1843619 (MCV 1,5/ 3-G-3,81); Supplier1 (none) -> Farnell: 3704828
- J3: Manufacturer (none) -> Phoenix: 1803426 (MCV 1,5/ 2-G-3,81); Supplier1 (none) -> Farnell: 3913077
- J4: renamed from J2; Manufacturer (none) -> Phoenix: 1803439 (MCV 1,5/ 3-G-3,81); Supplier1 (none) -> Farnell: 3913089
- R1: renamed from R8; footprint Resistor_THT:R_Axial_DIN0204_L3.6mm_D1.6mm_P5.08mm_Horizontal -> Resistor_THT:R_Axial_DIN0204_L3.6mm_D1.6mm_P7.62mm_Horizontal; Manufacturer Multicomp:MF12 20K -> Multicomp: MF12 15K; Supplier1 Farnell:9342796 -> Farnell: 9342630
- R13: renamed from R7; Manufacturer TE Connectivity:LR1F3R9 -> TE Connectivity: LR1F3R9; Supplier1 Farnell:2330141 -> Farnell: 2330141
- R14: renamed from R10; Manufacturer TE Connectivity:LR1F10R -> TE Connectivity: LR1F10R; Supplier1 Farnell:2329993 -> Farnell: 2329993
- R2: renamed from R11; footprint Resistor_THT:R_Axial_DIN0204_L3.6mm_D1.6mm_P5.08mm_Horizontal -> Resistor_THT:R_Axial_DIN0204_L3.6mm_D1.6mm_P7.62mm_Horizontal; Manufacturer Multicomp:MF12 20K -> Multicomp: MF12 47K; Supplier1 Farnell:9342796 -> Farnell: 9343261
- R3: renamed from R12; footprint Resistor_THT:R_Axial_DIN0204_L3.6mm_D1.6mm_P5.08mm_Horizontal -> Resistor_THT:R_Axial_DIN0204_L3.6mm_D1.6mm_P7.62mm_Horizontal; Manufacturer Multicomp:MF12 20K -> Multicomp: MF12 30K; Supplier1 Farnell:9342796 -> Farnell: 9343008
- R4: renamed from R13; footprint Resistor_THT:R_Axial_DIN0204_L3.6mm_D1.6mm_P5.08mm_Horizontal -> Resistor_THT:R_Axial_DIN0207_L6.3mm_D2.5mm_P10.16mm_Horizontal; Manufacturer Multicomp:MF12 20K -> Multicomp: MF25 10K; Power 1/8 -> 1/4; Supplier1 Farnell:9342796 -> Farnell: 9341110
- R9: Manufacturer TE Connectivity:LR1F3R9 -> TE Connectivity: LR1F3R9; Supplier1 Farnell:2330141 -> Farnell: 2330141
- renumbered J4 to J1, MK3 to MK2, MK2 to MK3, R4 to R10, R6 to R12
Connections:
- net +pwvs: now also D2.1 (K); no longer J1.1 (Pin_1)
- net -pwvs: now also C14.2, C15.2, C16.2, D4.2 (A); no longer C2.2
- net GNDD: now also C14.1, C2.2, J3.1 (Pin_1), C15.1, C16.1, R11.2; no longer C14.2, C2.1, J3.2 (Pin_2)
- net input: now also R6.2, R7.2; no longer C6.2
- net out: now also J3.2 (Pin_2); no longer J3.1 (Pin_1)
- net preout: now also D4.1 (K)
- net sgnd: now also R5.1, C5.2, R11.1, R7.1; no longer R5.2
- net mute: now reaches C1.1, R1.2, U1.10 (MUTE)
- net at U1.3 (+): now also C6.1, R5.2; no longer R5.1
- net stby: now reaches R3.2, U1.9 (STBY)
- net stby: now also C2.1; no longer C14.1
- net at D1.1 (K), R2.1, R3.1: now also J1.2 (Pin_2); no longer D2.2 (A), R4.2
- new net: C5.1, C6.2, R6.1
- new net: D2.2 (A), J1.1 (Pin_1), R4.2
Other:
- note added: "0.68 SHP"
- note added: "4.02 HP"
- note added: "7.2M LP"
- note added: "Matching connector:\nManufacturer: Molex 16-02-0082\nSupplier1: Farnell: 1756731\nManufactuer: Molex 50-57-9004\nSupplier1: Farnell: 1756895"
- note added: "Matching connector:\nManufacturer: Phoenix 1826979 (MCVW 1,5/ 2-ST-3,81)\nSupplier1: Farnell: 3705080"
- note added: "Matching connector:\nManufacturer: Phoenix 1826982 (MCVW 1,5/ 3-ST-3,81)\nSupplier1: Farnell: 3705092"
- note added: "Matching connector:\nManufacturer: Phoenix 1862865 (MCVW 1,5/ 3-ST-3,5)\nSupplier1: Farnell: 5089165"
- note removed: "1.32 HP"
- note removed: "1.44 SHP"
- moved on the sheet: C6, C7, D2, J1, J2, J3, LOGO1, LOGO2, MK1, MK2, MK3, MK4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

Commit message: WIP: Component pad editing.
Signed-off-by: Nenad Radulovic <nenad.b.radulovic@gmail.com>
Parts:
- added NT1: Net-Tie_2, NetTie:NetTie-2_SMD_Pad2.0mm, symbol Device:Net-Tie_2
- C11, C14: Supplier1 Farnel: 2346272 -> Farnell: 2346272
- C7: Supplier1 Farnel: 2346252 -> Farnell: 2346252
- D2: Manufacturer ON Semuconductor: BZX79C15 -> ON Semiconductor: BZX79C15
- R10: Manufacturer TE Connectivity:LR1F499R -> TE Connectivity: LR1F499R; Supplier1 Farnell:2330163 -> Farnell: 2330163
- R12: Supplier1 Farnell:2330007 -> Farnell: 2330007
- R5, R7: Manufacturer TE Connectivity:LR1F12K -> TE Connectivity: LR1F12K; Supplier1 Farnell:2330007 -> Farnell: 2330007
- U1: Supplier1 Farnell:1366582 -> Farnell: 1366582
Connections:
- net GNDD: now also NT1.2; no longer C10.2, C11.2, C12.2, C13.2, C14.1, C15.1, C16.1, C9.2, J2.3 (Pin_3), J3.1 (Pin_1), J4.2 (Pin_2), R11.2
- new net GNDPWR: C10.2, C11.2, C12.2, C13.2, C14.1, C15.1, C16.1, C9.2, J2.3 (Pin_3), J3.1 (Pin_1), J4.2 (Pin_2), NT1.1, R11.2
Other:
- note added: "Place jumper on pins 1 & 2\nto enable the amplifier."
Changed lines of the file:
@@
 F 3 "http://www.farnell.com/datasheets/1761334.pdf" H 6000 3100 50  0001 C CNN
 F 4 "ST:TDA7293V" H 2100 600 50  0001 C CNN "Manufacturer"
-F 5 "Farnell:1366582" H 2100 600 50  0001 C CNN "Supplier1"
+F 5 "Farnell: 1366582" H 2100 600 50  0001 C CNN "Supplier1"
 	1    6000 3100
 	1    0    0    -1
@@
 F 4 "0.6W" H 4030 3595 50  0000 R CNN "Power"
 F 5 "MF" H 4030 3686 50  0000 R CNN "Type"
-F 6 "TE Connectivity:LR1F12K" H 4100 3550 50  0001 C CNN "Manufacturer"
-F 7 "Farnell:2330007" H 4100 3550 50  0001 C CNN "Supplier1"
+F 6 "TE Connectivity: LR1F12K" H 4100 3550 50  0001 C CNN "Manufacturer"
+F 7 "Farnell: 2330007" H 4100 3550 50  0001 C CNN "Supplier1"
 	1    4100 3550
 	-1   0    0    1
@@
 	1    0    0    -1
 $EndComp
-Wire Wire Line
-	1600 6500 1900 6500
 Text Notes 6450 5350 0    50   ~ 0
 Return to supply bypass \ncapacitor ground
@@
 F 4 "10V" V 3745 3200 50  0000 C CNN "Voltage"
 F 5 "Rybicon:10YXJ470M6.3X11 " V 3400 3200 50  0001 C CNN "Manufacturer"
-F 6 "Farnel: 2346252" V 3400 3200 50  0001 C CNN "Supplier1"
+F 6 "Farnell: 2346252" V 3400 3200 50  0001 C CNN "Supplier1"
 	1    3400 3200
 	0    1    1    0
@@
 F 4 "0.6W" V 4097 3200 50  0000 C CNN "Power"
 F 5 "MF" V 4188 3200 50  0000 C CNN "Type"
-F 6 "TE Connectivity:LR1F499R" V 3800 3200 50  0001 C CNN "Manufacturer"
-F 7 "Farnell:2330163" V 3800 3200 50  0001 C CNN "Supplier1"
+F 6 "TE Connectivity: LR1F499R" V 3800 3200 50  0001 C CNN "Manufacturer"
+F 7 "Farnell: 2330163" V 3800 3200 50  0001 C CNN "Supplier1"
 	1    3800 3200
 	0    1    1    0
@@
 F 5 "MF" H 4770 3414 50  0000 L CNN "Type"
 F 6 "TE Connectivity:LR1F12K" H 4700 3550 50  0001 C CNN "Manufacturer"
-F 7 "Farnell:2330007" H 4700 3550 50  0001 C CNN "Supplier1"
+F 7 "Farnell: 2330007" H 4700 3550 50  0001 C CNN "Supplier1"
 	1    4700 3550
 	1    0    0    -1
@@
 F 4 "50V" H 2082 6159 50  0000 R CNN "Voltage"
 F 5 "Rybicon: 50YXJ2200M16X35.5" V 2200 6250 50  0001 C CNN "Manufacturer"
-F 6 "Farnel: 2346272" V 2200 6250 50  0001 C CNN "Supplier1"
+F 6 "Farnell: 2346272" V 2200 6250 50  0001 C CNN "Supplier1"
 	1    2200 6250
 	-1   0    0    -1
@@
 L power:GNDD #PWR012
 U 1 1 5C76C62A
-P 1900 6600
-F 0 "#PWR012" H 1900 6350 50  0001 C CNN
-F 1 "GNDD" H 1904 6445 50  0000 C CNN
-F 2 "" H 1900 6600 50  0001 C CNN
-F 3 "" H 1900 6600 50  0001 C CNN
-	1    1900 6600
-	1    0    0    -1
-$EndComp
-Wire Wire Line
-	1900 6600 1900 6500
-Connection ~ 1900 6500
-Wire Wire Line
-	1900 6500 2200 6500
+P 5150 5300
+F 0 "#PWR012" H 5150 5050 50  0001 C CNN
+F 1 "GNDD" V 5154 5190 50  0000 R CNN
+F 2 "" H 5150 5300 50  0001 C CNN
+F 3 "" H 5150 5300 50  0001 C CNN
+	1    5150 5300
+	0    -1   -1   0
+$EndComp
 Wire Wire Line
 	8800 3500 8800 1500
@@
 F 2 "Diode_THT:D_DO-35_SOD27_P7.62mm_Horizontal" H 10000 1150 50  0001 C CNN
 F 3 "http://www.farnell.com/datasheets/2299521.pdf" H 10000 1150 50  0001 C CNN
-F 4 "ON Semuconductor: BZX79C15" V 10000 1150 50  0001 C CNN "Manufacturer"
+F 4 "ON Semiconductor: BZX79C15" V 10000 1150 50  0001 C CNN "Manufacturer"
 F 5 "Farnell: 1467595" V 10000 1150 50  0001 C CNN "Supplier1"
 	1    10000 1150
@@
 F 4 "0.6W" H 2380 2995 50  0000 R CNN "Power"
 F 5 "MF" H 2380 3086 50  0000 R CNN "Type"
-F 6 "TE Connectivity:LR1F12K" H 2450 2950 50  0001 C CNN "Manufacturer"
-F 7 "Farnell:2330007" H 2450 2950 50  0001 C CNN "Supplier1"
+F 6 "TE Connectivity: LR1F12K" H 2450 2950 50  0001 C CNN "Manufacturer"
+F 7 "Farnell: 2330007" H 2450 2950 50  0001 C CNN "Supplier1"
 	1    2450 2950
 	-1   0    0    1
@@
 F 4 "50V" H 2082 6659 50  0000 R CNN "Voltage"
 F 5 "Rybicon: 50YXJ2200M16X35.5" V 2200 6750 50  0001 C CNN "Manufacturer"
-F 6 "Farnel: 2346272" V 2200 6750 50  0001 C CNN "Supplier1"
+F 6 "Farnell: 2346272" V 2200 6750 50  0001 C CNN "Supplier1"
 	1    2200 6750
 	-1   0    0    -1
@@
 Text Notes 2950 2300 0    50   ~ 0
 7.2M LP
-Text Notes 9450 2550 0    50   ~ 0
+Text Notes 9450 2600 0    50   ~ 0
 Matching connector:\nManufacturer: Molex 16-02-0082\nSupplier1: Farnell: 1756731\nManufactuer: Molex 50-57-9004\nSupplier1: Farnell: 1756895
 Text Notes 1550 1600 0    50   ~ 0
@@
 Text Label 6500 1600 0    50   ~ 0
 stby
+$Comp
+L Device:Net-Tie_2 NT1
+U 1 1 5C55F742
+P 4850 5300
+F 0 "NT1" H 4850 5478 50  0000 C CNN
+F 1 "Net-Tie_2" H 4850 5387 50  0000 C CNN
+F 2 "NetTie:NetTie-2_SMD_Pad2.0mm" H 4850 5300 50  0001 C CNN
+F 3 "~" H 4850 5300 50  0001 C CNN
+	1    4850 5300
+	1    0    0    -1
+$EndComp
+$Comp
+L power:GNDPWR #PWR013
+U 1 1 5C55FC9C
+P 4750 5300
+F 0 "#PWR013" H 4750 5100 50  0001 C CNN
+F 1 "GNDPWR" V 4754 5191 50  0000 R CNN
+F 2 "" H 4750 5250 50  0001 C CNN
+F 3 "" H 4750 5250 50  0001 C CNN
+	1    4750 5300
+	0    1    1    0
+$EndComp
+Wire Wire Line
+	1600 6500 2200 6500
+Wire Wire Line
+	4950 5300 5050 5300
+$Comp
+L power:PWR_FLAG #FLG0101
+U 1 1 5C56B7AF
+P 5050 5300
+F 0 "#FLG0101" H 5050 5375 50  0001 C CNN
+F 1 "PWR_FLAG" H 5050 5474 50  0000 C CNN
+F 2 "" H 5050 5300 50  0001 C CNN
+F 3 "~" H 5050 5300 50  0001 C CNN
+	1    5050 5300
+	1    0    0    -1
+$EndComp
+Connection ~ 5050 5300
+Wire Wire Line
+	5050 5300 5150 5300
+Wire Notes Line
+	8550 5100 10850 5100
+Wire Notes Line
+	10850 5450 8550 5450
+Wire Notes Line
+	8550 5450 8550 5100
+Wire Notes Line
+	10850 3100 9800 3100
+Wire Notes Line
+	10850 3100 10850 5450
+Wire Notes Line
+	9400 2150 10800 2150
+Wire Notes Line
+	10800 2150 10800 2650
+Wire Notes Line
+	10800 2650 9400 2650
+Wire Notes Line
+	9400 2650 9400 1600
+Wire Notes Line
+	4400 7300 6700 7300
+Wire Notes Line
+	6700 7300 6700 7650
+Wire Notes Line
+	4400 7650 4400 7300
+Wire Notes Line
+	1000 7650 1000 6700
+Wire Notes Line
+	1000 7650 6700 7650
+Wire Notes Line
+	1500 1300 3750 1300
+Wire Notes Line
+	3750 1300 3750 1650
+Wire Notes Line
+	3750 1650 1500 1650
+Wire Notes Line
+	1500 1300 1500 2600
+Wire Notes Line
+	9450 1200 9600 1200
+Wire Notes Line
+	9600 1200 9600 1300
+Wire Notes Line
+	9600 1300 9450 1300
+Text Notes 8700 750  0    50   ~ 0
+Place jumper on pins 1 & 2\nto enable the amplifier.
+Wire Notes Line
+	8650 550  9850 550
+Wire Notes Line
+	9850 800  8650 800
+Wire Notes Line
+	8650 800  8650 550
+Wire Notes Line
+	9850 1200 9650 1200
+Wire Notes Line
+	9850 550  9850 1200
 $EndSCHEMATC
