File: parvus_amp/parvus_amp.sch (KiCad schematic (older format))
At the start: 45 parts, among them J1 ctrl, J2 input, J3 output, J4 power, U1 TDA7293

Commit message: Added some Mouser identifiers
Parts:
- C10: Supplier2 (none) -> Mouser: 581-SR211C104KAR
- C12, C15: Supplier2 (none) -> Mouser: 505-MKS0C032200C00KS
- C13, C16: Supplier2 (none) -> Mouser: 505-MKS02.022/63/10
- C5: Supplier2 (none) -> Mouser: 80-C315C221K2G
- C8: Supplier2 (none) -> Mouser: 80-C315C339D2G
- C9: Supplier2 (none) -> Mouser: 505-MKS02.1/63/10
- D1: Supplier2 (none) -> Mouser: 512-1N4148TA
- D2: Supplier2 (none) -> Mouser: 512-BZX79C15
- D3, D4: Supplier2 (none) -> Mouser: 863-1N5404RLG
- J2: Supplier2 (none) -> Mouser: 651-1843619
- J3: Supplier2 (none) -> Mouser: 651-1803426
- J4: Supplier2 (none) -> Mouser: 651-1803439
- R1: Manufacturer Multicomp: MF12 15K -> (none); Manufacturer1 (none) -> Multicomp: MF12 15K; Manufacturer2 (none) -> Yageo: CFR-25JR-52-15K; Supplier2 (none) -> Mouser: 603-CFR-25JR-5215K
- R10: Supplier2 (none) -> Mouser: 279-LR1F499R
- R11, R14: Supplier2 (none) -> Mouser: 279-LR1F10R
- R12: Manufacturer TE Connectivity:LR1F12K -> TE Connectivity: LR1F12K; Supplier2 (none) -> Mouser: 279-LR1F12K
- R13, R9: Manufacturer TE Connectivity: LR1F3R9 -> (none); Manufacturer1 (none) -> TE Connectivity: LR1F3R9; Manufacturer2 (none) -> Vishay/BC Components: PR01000103908JR500; Supplier2 (none) -> Mouser: 594-5073NW3R900J
- R2: Manufacturer Multicomp: MF12 47K -> (none); Manufacturer1 (none) -> Multicomp: MF12 47K; Manufacturer2 (none) -> Yageo: CFR-25JR-52-47K; Supplier2 (none) -> Mouser: 603-CFR-25JR-5247K
- R3: Manufacturer Multicomp: MF12 30K -> (none); Manufacturer1 (none) -> Multicomp: MF12 30K; Manufacturer2 (none) -> Yageo: CFR-25JR-52-30K; Supplier2 (none) -> Mouser: 603-CFR-25JR-52-30K
- R4: Manufacturer Multicomp: MF25 10K -> (none); Manufacturer1 (none) -> Multicomp: MF25 10K; Manufacturer2 (none) -> Yageo: CFR-25JR-52-10K; Supplier2 (none) -> Mouser: 603-CFR-25JR-5210K
- R5, R7: Supplier2 (none) -> Mouser: 279-LR1F12K
- R6: Supplier2 (none) -> Mouser: 279-LR1F100R
- U1: Supplier2 (none) -> Mouser: 511-TDA7293V
Changed lines of the file:
@@
 F 4 "ST:TDA7293V" H 2100 600 50  0001 C CNN "Manufacturer"
 F 5 "Farnell: 1366582" H 2100 600 50  0001 C CNN "Supplier1"
+F 6 "Mouser: 511-TDA7293V" H 6000 3100 50  0001 C CNN "Supplier2"
 	1    6000 3100
 	1    0    0    -1
@@
 F 6 "Kemet: C315C339D2G5TA" V 5300 3550 50  0001 C CNN "Manufacturer"
 F 7 "Farnell: 2819636" V 5300 3550 50  0001 C CNN "Supplier1"
+F 8 "Mouser: 80-C315C339D2G" H 0   0   50  0001 C CNN "Supplier2"
 	1    5300 3550
 	1    0    0    -1
@@
 F 4 "0.6W" H 7670 4005 50  0000 L CNN "Power"
 F 5 "MF" H 7670 3914 50  0000 L CNN "Type"
-F 6 "TE Connectivity: LR1F3R9" H 7600 4050 50  0001 C CNN "Manufacturer"
-F 7 "Farnell: 2330141" H 7600 4050 50  0001 C CNN "Supplier1"
+F 6 "TE Connectivity: LR1F3R9" H 7600 4050 50  0001 C CNN "Manufacturer1"
+F 7 "Vishay/BC Components: PR01000103908JR500" H 7600 4050 50  0001 C CNN "Manufacturer2"
+F 8 "Farnell: 2330141" H 7600 4050 50  0001 C CNN "Supplier1"
+F 9 "Mouser: 594-5073NW3R900J" H 0   0   50  0001 C CNN "Supplier2"
 	1    7600 4050
 	1    0    0    -1
@@
 F 6 "WIMA: MKS0C031000C00KSSD" H 2700 600 50  0001 C CNN "Manufacturer"
 F 7 "Farnell: 1006004" H 2700 600 50  0001 C CNN "Supplier1"
+F 8 "Mouser: 505-MKS02.1/63/10 " H 0   0   50  0001 C CNN "Supplier2"
 	1    7600 4450
 	1    0    0    -1
@@
 F 4 "ON Semiconductor: 1N5404RL" V 6800 2650 50  0001 C CNN "Manufacturer"
 F 5 "Farnell: 9556141" V 6800 2650 50  0001 C CNN "Supplier1"
+F 6 "Mouser: 863-1N5404RLG" H 0   0   50  0001 C CNN "Supplier2"
 	1    6800 2650
 	0    -1   1    0
@@
 F 6 "TE Connectivity: LR1F12K" H 4100 3550 50  0001 C CNN "Manufacturer"
 F 7 "Farnell: 2330007" H 4100 3550 50  0001 C CNN "Supplier1"
+F 8 "Mouser: 279-LR1F12K" H 0   0   50  0001 C CNN "Supplier2"
 	1    4100 3550
 	-1   0    0    1
@@
 F 6 "AVX: SR211C104KAR" H 2700 600 50  0001 C CNN "Manufacturer"
 F 7 "Farnell: 1100408" H 2700 600 50  0001 C CNN "Supplier1"
+F 8 "Mouser: 581-SR211C104KAR" H 0   0   50  0001 C CNN "Supplier2"
 	1    8100 4450
 	1    0    0    -1
@@
 F 6 "WIMA: MKS0C032200C00KSSD" H 2800 6250 50  0001 C CNN "Manufacturer"
 F 7 "Farnell: 1890123" H 2800 6250 50  0001 C CNN "Supplier1"
+F 8 "Mouser: 505-MKS0C032200C00KS" H 0   0   50  0001 C CNN "Supplier2"
 	1    2800 6250
 	1    0    0    -1
@@
 F 4 "1/8" V 8547 1600 50  0000 C CNN "Power"
 F 5 "C" V 8638 1600 50  0000 C CNN "Type"
-F 6 "Multicomp: MF12 30K" V 8250 1600 50  0001 C CNN "Manufacturer"
+F 6 "" V 8250 1600 50  0001 C CNN "Manufacturer"
 F 7 "Farnell: 9343008" V 8250 1600 50  0001 C CNN "Supplier1"
+F 8 "Multicomp: MF12 30K" H 0   0   50  0001 C CNN "Manufacturer1"
+F 9 "Yageo: CFR-25JR-52-30K" H 0   0   50  0001 C CNN "Manufacturer2"
+F 10 "Mouser: 603-CFR-25JR-52-30K" H 0   0   50  0001 C CNN "Supplier2"
 	1    8250 1600
 	0    1    1    0
@@
 F 6 "TE Connectivity: LR1F499R" V 3800 3200 50  0001 C CNN "Manufacturer"
 F 7 "Farnell: 2330163" V 3800 3200 50  0001 C CNN "Supplier1"
+F 8 "Mouser: 279-LR1F499R" H 0   0   50  0001 C CNN "Supplier2"
 	1    3800 3200
 	0    1    1    0
@@
 F 4 "0.6W" H 4770 3505 50  0000 L CNN "Power"
 F 5 "MF" H 4770 3414 50  0000 L CNN "Type"
-F 6 "TE Connectivity:LR1F12K" H 4700 3550 50  0001 C CNN "Manufacturer"
+F 6 "TE Connectivity: LR1F12K" H 4700 3550 50  0001 C CNN "Manufacturer"
 F 7 "Farnell: 2330007" H 4700 3550 50  0001 C CNN "Supplier1"
+F 8 "Mouser: 279-LR1F12K" H 0   0   50  0001 C CNN "Supplier2"
 	1    4700 3550
 	1    0    0    -1
@@
 F 4 "0.6W" V 8200 3100 50  0000 C CNN "Power"
 F 5 "MF" V 8300 3100 50  0000 C CNN "Type"
-F 6 "TE Connectivity: LR1F3R9" H 7850 3100 50  0001 C CNN "Manufacturer"
+F 6 "" H 7850 3100 50  0001 C CNN "Manufacturer"
 F 7 "Farnell: 2330141" H 7850 3100 50  0001 C CNN "Supplier1"
+F 8 "Mouser: 594-5073NW3R900J" H 0   0   50  0001 C CNN "Supplier2"
+F 9 "TE Connectivity: LR1F3R9" H 0   0   50  0001 C CNN "Manufacturer1"
+F 10 "Vishay/BC Components: PR01000103908JR500" H 0   0   50  0001 C CNN "Manufacturer2"
 	1    7850 3100
 	0    1    1    0
@@
 F 6 "TE Connectivity: LR1F10R" H 8100 4050 50  0001 C CNN "Manufacturer"
 F 7 "Farnell: 2329993" H 8100 4050 50  0001 C CNN "Supplier1"
+F 8 "Mouser: 279-LR1F10R" H 0   0   50  0001 C CNN "Supplier2"
 	1    8100 4050
 	1    0    0    -1
@@
 F 4 "1/8" V 7600 1300 50  0000 C CNN "Power"
 F 5 "C" V 7700 1300 50  0000 C CNN "Type"
-F 6 "Multicomp: MF12 47K" V 7850 1300 50  0001 C CNN "Manufacturer"
+F 6 "" V 7850 1300 50  0001 C CNN "Manufacturer"
 F 7 "Farnell: 9343261" V 7850 1300 50  0001 C CNN "Supplier1"
+F 8 "Multicomp: MF12 47K" H 0   0   50  0001 C CNN "Manufacturer1"
+F 9 "Yageo: CFR-25JR-52-47K" H 0   0   50  0001 C CNN "Manufacturer2"
+F 10 "Mouser: 603-CFR-25JR-5247K" H 0   0   50  0001 C CNN "Supplier2"
 	1    7850 1300
 	0    1    1    0
@@
 F 4 "ON Semiconductor: 1N4148TA" H 8250 1000 50  0001 C CNN "Manufacturer"
 F 5 "Farnell: 2322485" H 8250 1000 50  0001 C CNN "Supplier1"
+F 6 "Mouser: 512-1N4148TA" H 0   0   50  0001 C CNN "Supplier2"
 	1    8250 1000
 	-1   0    0    1
@@
 F 4 "Phoenix: 1803439 (MCV 1,5/ 3-G-3,81)" H 1000 6500 50  0001 C CNN "Manufacturer"
 F 5 "Farnell: 3913089" H 1000 6500 50  0001 C CNN "Supplier1"
+F 6 "Mouser: 651-1803439" H 0   0   50  0001 C CNN "Supplier2"
 	1    1000 6500
 	-1   0    0    -1
@@
 F 4 "Phoenix: 1843619 (MCV 1,5/ 3-G-3,81)" H 1550 2800 50  0001 C CNN "Manufacturer"
 F 5 "Farnell: 3704828" H 1550 2800 50  0001 C CNN "Supplier1"
+F 6 "Mouser: 651-1843619" H 0   0   50  0001 C CNN "Supplier2"
 	1    1550 2800
 	-1   0    0    -1
@@
 F 4 "Phoenix: 1803426 (MCV 1,5/ 2-G-3,81)" H 9400 3000 50  0001 C CNN "Manufacturer"
 F 5 "Farnell: 3913077" H 9400 3000 50  0001 C CNN "Supplier1"
+F 6 "Mouser: 651-1803426" H 0   0   50  0001 C CNN "Supplier2"
 	1    9400 3000
 	1    0    0    -1
@@
 F 6 "WIMA: MKS0C022200B00KSSD" H 3400 6250 50  0001 C CNN "Manufacturer"
 F 7 "Farnell: 1006001" H 3400 6250 50  0001 C CNN "Supplier1"
+F 8 "Mouser: 505-MKS02.022/63/10" H 0   0   50  0001 C CNN "Supplier2"
 	1    3400 6250
 	1    0    0    -1
@@
 F 4 "1/4" H 9930 1695 50  0000 R CNN "Power"
 F 5 "C" H 9930 1786 50  0000 R CNN "Type"
-F 6 "Multicomp: MF25 10K" V 10000 1650 50  0001 C CNN "Manufacturer"
+F 6 "" V 10000 1650 50  0001 C CNN "Manufacturer"
 F 7 "Farnell: 9341110" V 10000 1650 50  0001 C CNN "Supplier1"
+F 8 "Multicomp: MF25 10K" H 0   0   50  0001 C CNN "Manufacturer1"
+F 9 "Yageo: CFR-25JR-52-10K" H 0   0   50  0001 C CNN "Manufacturer2"
+F 10 "Mouser: 603-CFR-25JR-5210K" H 0   0   50  0001 C CNN "Supplier2"
 	1    10000 1650
 	-1   0    0    1
@@
 F 4 "1/8" V 7143 1300 50  0000 C CNN "Power"
 F 5 "C" V 7234 1300 50  0000 C CNN "Type"
-F 6 "Multicomp: MF12 15K" V 7350 1300 50  0001 C CNN "Manufacturer"
+F 6 "" V 7350 1300 50  0001 C CNN "Manufacturer"
 F 7 "Farnell: 9342630" V 7350 1300 50  0001 C CNN "Supplier1"
+F 8 "Multicomp: MF12 15K" H 0   0   50  0001 C CNN "Manufacturer1"
+F 9 "Yageo: CFR-25JR-52-15K" H 0   0   50  0001 C CNN "Manufacturer2"
+F 10 "Mouser: 603-CFR-25JR-5215K" H 0   0   50  0001 C CNN "Supplier2"
 	1    7350 1300
 	0    1    1    0
@@
 F 4 "ON Semiconductor: BZX79C15" V 10000 1150 50  0001 C CNN "Manufacturer"
 F 5 "Farnell: 1467595" V 10000 1150 50  0001 C CNN "Supplier1"
+F 6 "Mouser: 512-BZX79C15" H 0   0   50  0001 C CNN "Supplier2"
 	1    10000 1150
 	0    1    1    0
@@
 F 6 "Kemet: C315C221K2G5TA" V 2950 2950 50  0001 C CNN "Manufacturer"
 F 7 "Farnell: 2819626" V 2950 2950 50  0001 C CNN "Supplier1"
+F 8 "Mouser: 80-C315C221K2G" H 0   0   50  0001 C CNN "Supplier2"
 	1    2950 2950
 	1    0    0    -1
@@
 F 6 "TE Connectivity: LR1F12K" H 2450 2950 50  0001 C CNN "Manufacturer"
 F 7 "Farnell: 2330007" H 2450 2950 50  0001 C CNN "Supplier1"
+F 8 "Mouser: 279-LR1F12K" H 0   0   50  0001 C CNN "Supplier2"
 	1    2450 2950
 	-1   0    0    1
@@
 F 6 "TE Connectivity: LR1F10R" H 2450 3450 50  0001 C CNN "Manufacturer"
 F 7 "Farnell: 2329993" H 2450 3450 50  0001 C CNN "Supplier1"
+F 8 "Mouser: 279-LR1F10R" H 0   0   50  0001 C CNN "Supplier2"
 	1    2450 3450
 	1    0    0    -1
@@
 F 4 "ON Semiconductor: 1N5404RL" V 6800 4150 50  0001 C CNN "Manufacturer"
 F 5 "Farnell: 9556141" V 6800 4150 50  0001 C CNN "Supplier1"
+F 6 "Mouser: 863-1N5404RLG" H 0   0   50  0001 C CNN "Supplier2"
 	1    6800 4150
 	0    -1   1    0
@@
 F 6 "WIMA: MKS0C022200B00KSSD" H 3400 6750 50  0001 C CNN "Manufacturer"
 F 7 "Farnell: 1006001" H 3400 6750 50  0001 C CNN "Supplier1"
+F 8 "Mouser: 505-MKS02.022/63/10" H 0   0   50  0001 C CNN "Supplier2"
 	1    3400 6750
 	1    0    0    -1
@@
 F 6 "WIMA: MKS0C032200C00KSSD" H 2800 6750 50  0001 C CNN "Manufacturer"
 F 7 "Farnell: 1890123" H 2800 6750 50  0001 C CNN "Supplier1"
+F 8 "Mouser: 505-MKS0C032200C00KS" H 0   0   50  0001 C CNN "Supplier2"
 	1    2800 6750
 	1    0    0    -1
@@
 F 6 "TE Connectivity: LR1F100R" V 2700 2700 50  0001 C CNN "Manufacturer"
 F 7 "Farnell: 2329988" V 2700 2700 50  0001 C CNN "Supplier1"
+F 8 "Mouser: 279-LR1F100R" H 0   0   50  0001 C CNN "Supplier2"
 	1    2700 2700
 	0    1    1    0
