File: parvus_amp/parvus_amp.sch (KiCad schematic (older format))
At the start: 45 parts, among them J1 ctrl, J2 input, J3 output, J4 power, U1 TDA7293

Commit message: Modified st-by/mute circuit values to accomodate control circuitry in PSU.
Signed-off-by: Nenad Radulovic <nenad.b.radulovic@gmail.com>
Parts:
- R1: value 15k -> 2k; Manufacturer2 Yageo: CFR-25JR-52-15K -> Yageo: CFR-25JB-52-2K; Supplier2 Mouser: 603-CFR-25JR-5215K -> Mouser: 603-CFR-25JB-52-2K
- R2: value 47k -> 18k; Manufacturer1 Multicomp: MF12 47K -> Multicomp: MF12 18K; Manufacturer2 Yageo: CFR-25JR-52-47K -> Yageo: CFR-12JB-52-18K; Power 1/8 -> 1/4; Supplier1 Farnell: 9343261 -> Farnell: 9342745; Supplier2 Mouser: 603-CFR-25JR-5247K -> Mouser: 603-CFR-12JB-52-18K
- R3: value 30k -> 10k; Manufacturer2 Yageo: CFR-25JR-52-30K -> Yageo: CFR-12JB-52-10K; Supplier2 Mouser: 603-CFR-25JR-52-30K -> Mouser: 603-CFR-12JB-52-10K
Changed lines of the file:
@@
 P 8250 1600
 F 0 "R3" V 8365 1600 50  0000 C CNN
-F 1 "30k" V 8456 1600 50  0000 C CNN
+F 1 "10k" V 8456 1600 50  0000 C CNN
 F 2 "Resistor_THT:R_Axial_DIN0204_L3.6mm_D1.6mm_P7.62mm_Horizontal" V 8180 1600 50  0001 C CNN
 F 3 "http://www.farnell.com/datasheets/1716726.pdf" H 8250 1600 50  0001 C CNN
@@
 F 6 "Farnell: 9343008" V 8250 1600 50  0001 C CNN "Supplier1"
 F 7 "Multicomp: MF12 30K" H 0   0   50  0001 C CNN "Manufacturer1"
-F 8 "Mouser: 603-CFR-25JR-52-30K" H 0   0   50  0001 C CNN "Supplier2"
-F 9 "Yageo: CFR-25JR-52-30K" H 0   0   50  0001 C CNN "Manufacturer2"
+F 8 "Mouser: 603-CFR-12JB-52-10K" H 0   0   50  0001 C CNN "Supplier2"
+F 9 "Yageo: CFR-12JB-52-10K" H 0   0   50  0001 C CNN "Manufacturer2"
 	1    8250 1600
 	0    1    1    0
@@
 P 7850 1300
 F 0 "R2" V 7400 1300 50  0000 C CNN
-F 1 "47k" V 7500 1300 50  0000 C CNN
+F 1 "18k" V 7500 1300 50  0000 C CNN
 F 2 "Resistor_THT:R_Axial_DIN0204_L3.6mm_D1.6mm_P7.62mm_Horizontal" V 7780 1300 50  0001 C CNN
 F 3 "http://www.farnell.com/datasheets/1716726.pdf" H 7850 1300 50  0001 C CNN
-F 4 "1/8" V 7600 1300 50  0000 C CNN "Power"
+F 4 "1/4" V 7600 1300 50  0000 C CNN "Power"
 F 5 "C" V 7700 1300 50  0000 C CNN "Type"
-F 6 "Farnell: 9343261" V 7850 1300 50  0001 C CNN "Supplier1"
-F 7 "Multicomp: MF12 47K" H 0   0   50  0001 C CNN "Manufacturer1"
-F 8 "Mouser: 603-CFR-25JR-5247K" H 0   0   50  0001 C CNN "Supplier2"
-F 9 "Yageo: CFR-25JR-52-47K" H 0   0   50  0001 C CNN "Manufacturer2"
+F 6 "Farnell: 9342745" V 7850 1300 50  0001 C CNN "Supplier1"
+F 7 "Multicomp: MF12 18K" H 0   0   50  0001 C CNN "Manufacturer1"
+F 8 "Mouser: 603-CFR-12JB-52-18K" H 0   0   50  0001 C CNN "Supplier2"
+F 9 "Yageo: CFR-12JB-52-18K" H 0   0   50  0001 C CNN "Manufacturer2"
 	1    7850 1300
 	0    1    1    0
@@
 P 7350 1300
 F 0 "R1" V 6961 1300 50  0000 C CNN
-F 1 "15k" V 7052 1300 50  0000 C CNN
+F 1 "2k" V 7052 1300 50  0000 C CNN
 F 2 "Resistor_THT:R_Axial_DIN0204_L3.6mm_D1.6mm_P7.62mm_Horizontal" V 7280 1300 50  0001 C CNN
 F 3 "http://www.farnell.com/datasheets/1716726.pdf" H 7350 1300 50  0001 C CNN
@@
 F 6 "Farnell: 9342630" V 7350 1300 50  0001 C CNN "Supplier1"
 F 7 "Multicomp: MF12 15K" H 0   0   50  0001 C CNN "Manufacturer1"
-F 8 "Mouser: 603-CFR-25JR-5215K" H 0   0   50  0001 C CNN "Supplier2"
-F 9 "Yageo: CFR-25JR-52-15K" H 0   0   50  0001 C CNN "Manufacturer2"
+F 8 "Mouser: 603-CFR-25JB-52-2K" H 0   0   50  0001 C CNN "Supplier2"
+F 9 "Yageo: CFR-25JB-52-2K" H 0   0   50  0001 C CNN "Manufacturer2"
 	1    7350 1300
 	0    1    1    0
