File: parvus_amp/parvus_amp.kicad_pcb (KiCad board)
At the start: 2 copper layers, 70 x 54 mm, 45 parts, among them J1 ctrl, J2 input, J3 output, J4 power, U1 TDA7293

Commit message: Added text labels on silk screen.
Signed-off-by: Nenad Radulovic <nenad.b.radulovic@gmail.com>
Parts:
- moved LOGO2 63.2 mm to (91.5, 61.4)
Other:
- board text added: "-/PG/+ 24V"
- board text added: "190205"
- board text added: "44mm"
- board text added: "60mm"
- board text added: "PG/+ out"
- board text added: "PG/G/in"
- board text added: "REAL TIME CONSULTING"
- board text added: "parvus v1.0"
Changed lines of the file:
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@@
   (general
     (thickness 1.6)
-    (drawings 39)
+    (drawings 61)
     (tracks 175)
     (zones 0)
@@
   )
   (layers
-    (0 F.Cu signal hide)
-    (31 B.Cu signal hide)
+    (0 F.Cu signal)
+    (31 B.Cu signal)
     (32 B.Adhes user)
     (33 F.Adhes user)
     (34 B.Paste user)
     (35 F.Paste user)
-    (36 B.SilkS user hide)
+    (36 B.SilkS user)
     (37 F.SilkS user)
     (38 B.Mask user)
     (39 F.Mask user)
-    (40 Dwgs.User user hide)
-    (41 Cmts.User user hide)
-    (42 Eco1.User user hide)
-    (43 Eco2.User user hide)
+    (40 Dwgs.User user)
+    (41 Cmts.User user)
+    (42 Eco1.User user)
+    (43 Eco2.User user)
     (44 Edge.Cuts user)
-    (45 Margin user hide)
-    (46 B.CrtYd user hide)
-    (47 F.CrtYd user hide)
-    (48 B.Fab user hide)
-    (49 F.Fab user hide)
+    (45 Margin user)
+    (46 B.CrtYd user)
+    (47 F.CrtYd user)
+    (48 B.Fab user)
+    (49 F.Fab user)
   )
   (setup
@@
   )
   (module Symbol:OSHW-Logo2_7.3x6mm_SilkScreen (layer F.Cu)
-    (at 143.455 97.42)
+    (at 91.5 61.42)
     (descr "Open Source Hardware Symbol")
     (tags "Logo Symbol OSHW")
@@
     )
   )
+  (gr_text "PG/+\nout" (at 102.815 99.394) (layer B.SilkS)
+    (effects (font (size 1.5 1.5) (thickness 0.3)) (justify mirror))
+  )
+  (gr_line (start 102.18 81.36) (end 95.83 83.265) (layer B.SilkS) (width 0.2))
+  (gr_line (start 102.18 72.47) (end 102.18 81.36) (layer B.SilkS) (width 0.2))
+  (gr_text PG/G/in (at 104.085 76.915 270) (layer B.SilkS)
+    (effects (font (size 1.5 1.5) (thickness 0.3)) (justify mirror))
+  )
+  (gr_text "parvus\nv1.0" (at 132.025 84.535) (layer B.SilkS)
+    (effects (font (size 1.5 1.5) (thickness 0.3)) (justify mirror))
+  )
+  (gr_text 190205 (at 142.5 98.42) (layer F.Cu)
+    (effects (font (size 1.5 1.5) (thickness 0.3)))
+  )
+  (gr_text "REAL  TIME\nCONSULTING" (at 148.5 66.42) (layer F.Cu)
+    (effects (font (size 1.5 1.5) (thickness 0.3)))
+  )
+  (gr_text "-/PG/+\n24V" (at 115.5 99.394) (layer B.SilkS)
+    (effects (font (size 1.5 1.5) (thickness 0.3)) (justify mirror))
+  )
+  (gr_line (start 92.5 89.42) (end 93.5 90.42) (layer B.SilkS) (width 0.2))
+  (gr_line (start 92.5 89.42) (end 93.5 88.42) (layer B.SilkS) (width 0.2))
+  (gr_line (start 96.5 89.42) (end 92.5 89.42) (layer B.SilkS) (width 0.2))
+  (gr_line (start 144.5 97.42) (end 145.5 96.42) (layer B.SilkS) (width 0.2))
+  (gr_line (start 144.5 97.42) (end 143.5 96.42) (layer B.SilkS) (width 0.2))
+  (gr_line (start 144.5 93.42) (end 144.5 97.42) (layer B.SilkS) (width 0.2))
+  (gr_text 60mm (at 90.5 92.42 270) (layer B.SilkS)
+    (effects (font (size 1.5 1.5) (thickness 0.3)) (justify left mirror))
+  )
+  (gr_text 44mm (at 147.5 99.42) (layer B.SilkS)
+    (effects (font (size 1.5 1.5) (thickness 0.3)) (justify left mirror))
+  )
+  (gr_line (start 143.5 97.42) (end 148.5 97.42) (layer B.SilkS) (width 0.2))
+  (gr_line (start 92.5 93.42) (end 92.5 88.42) (layer B.SilkS) (width 0.2))
+  (gr_circle (center 152.5 53.42) (end 148.5 53.42) (layer B.SilkS) (width 0.2))
+  (gr_circle (center 152.5 97.42) (end 148.5 97.42) (layer B.SilkS) (width 0.2))
+  (gr_circle (center 92.5 97.42) (end 96.5 97.42) (layer B.SilkS) (width 0.2))
+  (gr_circle (center 92.5 53.42) (end 96.5 53.42) (layer B.SilkS) (width 0.2))
   (gr_line (start 114.88 86.948) (end 114.88 86.059) (layer F.SilkS) (width 0.4))
   (gr_line (start 112.34 86.948) (end 114.88 86.948) (layer F.SilkS) (width 0.4))
@@
     (polygon
       (pts
-        (xy 122.5 93.044) (xy 122.5 60.405) (xy 123.135 59.77) (xy 129.866 59.77) (xy 129.866 65.231)
+        (xy 122.5 93.044) (xy 122.5 60.913) (xy 123.008 60.405) (xy 129.866 60.405) (xy 129.866 65.231)
         (xy 131.39 66.755) (xy 131.39 93.044) (xy 130.755 93.679) (xy 123.135 93.679)
       )
@@
     (polygon
       (pts
-        (xy 130.374 59.77) (xy 140.28 59.77) (xy 140.915 60.405) (xy 140.915 64.85) (xy 140.28 65.485)
+        (xy 130.374 60.405) (xy 140.28 60.405) (xy 140.915 61.04) (xy 140.915 64.85) (xy 140.28 65.485)
         (xy 140.28 68.025) (xy 140.28 95.965) (xy 139.645 96.6) (xy 132.66 96.6) (xy 131.898 95.838)
         (xy 131.898 66.374) (xy 130.374 64.85)
@@
     (polygon
       (pts
-        (xy 123.135 96.6) (xy 122.5 95.965) (xy 122.5 60.405) (xy 123.77 59.77) (xy 140.28 59.77)
-        (xy 140.915 60.405) (xy 140.915 64.85) (xy 140.28 65.485) (xy 140.28 95.965) (xy 139.645 96.6)
+        (xy 123.135 96.6) (xy 122.5 95.965) (xy 122.5 61.04) (xy 123.135 60.405) (xy 140.28 60.405)
+        (xy 140.915 61.04) (xy 140.915 64.85) (xy 140.28 65.485) (xy 140.28 95.965) (xy 139.645 96.6)
       )
     )
@@
     (polygon
       (pts
-        (xy 121.865 89.615) (xy 111.705 89.615) (xy 111.07 88.98) (xy 111.07 62.31) (xy 111.705 61.675)
+        (xy 121.865 88.98) (xy 111.705 88.98) (xy 111.07 88.345) (xy 111.07 62.31) (xy 111.705 61.675)
         (xy 121.23 61.675) (xy 121.865 62.31)
       )
     )
+  )
+  (zone (net 1) (net_name GNDD) (layer F.Cu) (hatch edge 0.508)
+    (connect_pads yes (clearance 0.3))
+    (min_thickness 0.254)
+    (fill yes (arc_segments 16) (thermal_gap 0.508) (thermal_bridge_width 0.508))
+    (polygon
+      (pts
+        (xy 115.515 88.98) (xy 115.515 87.075) (xy 117.42 87.075) (xy 117.42 88.98)
+      )
+    )

Commit message: Adjusted NFB capacitor footprint and rest of Mouser IDs.
Signed-off-by: Nenad Radulovic <nenad.b.radulovic@gmail.com>
Parts:
- C7: footprint Capacitor_THT:CP_Radial_D6.3mm_P2.50mm -> Capacitor_THT:CP_Radial_D8.0mm_P3.50mm
- LOGO2: moved to B.Cu
- moved LOGO2 44.1 mm to (132.0, 78.8), turned to 180 degrees
- moved C7 1.27 mm to (95.2, 66.8)
- moved LOGO1 0.51 mm to (90.2, 65.5)
Routing:
- net /sgnd: track 100.4 -> 102.0 mm
- net Net-(C7-Pad1): track 9.15 -> 9.68 mm
Other:
- board text added: "Board grid origin: pin 8 of U1 component"
