File: parvus_psu/parvus_psu.sch (KiCad schematic (older format))
At the start: 30 parts, among them J1 tr_sec, J2 switch, J3 ac_input, J4 tr_pri, J5 left_power, J6 right_power

Commit message: Using 555 as AC detector.
Signed-off-by: Nenad Radulovic <nenad.b.radulovic@gmail.com>
Parts:
- added C?: 470n, Capacitor_THT:C_Rect_L7.2mm_W8.5mm_P5.00mm_FKP2_FKP2_MKS2_MKP2, symbol Device:C
- added D3, D4, D?: 1N4148, Diode_THT:D_DO-35_SOD27_P7.62mm_Horizontal, symbol Device:D
- added J?: left_power, Connector_PinHeader_2.54mm:PinHeader_1x04_P2.54mm_Vertical, symbol Connector_Generic:Conn_01x04
- added J?: left_power, Connector_PinHeader_2.54mm:PinHeader_1x04_P2.54mm_Vertical, symbol Connector_Generic:Conn_01x03
- added Q1: BC546B, Package_TO_SOT_THT:TO-92_Inline_Wide, symbol Device:Q_NPN_CBE
- added R6: 100k, Resistor_THT:R_Axial_DIN0207_L6.3mm_D2.5mm_P10.16mm_Horizontal, symbol Device:R
- added R7, R? (x3): 10k, Resistor_THT:R_Axial_DIN0207_L6.3mm_D2.5mm_P10.16mm_Horizontal, symbol Device:R
- added R9, R?: 47k, Resistor_THT:R_Axial_DIN0207_L6.3mm_D2.5mm_P10.16mm_Horizontal, symbol Device:R
- added U?: NE555, symbol Timer:NE555
Connections:
- wire segments 105 -> 160
- no-connect marks 0 -> 1
Other:
- moved on the sheet: MH1, MH2, MH3, MH4

Commit message: Finished schematic for AC detection circuit and clipping signaling.
Signed-off-by: Nenad Radulovic <nenad.b.radulovic@gmail.com>
Parts:
- removed C?: 470n, Capacitor_THT:C_Rect_L7.2mm_W8.5mm_P5.00mm_FKP2_FKP2_MKS2_MKP2, symbol Device:C
- removed D?: 1N4148, Diode_THT:D_DO-35_SOD27_P7.62mm_Horizontal, symbol Device:D
- removed R?: 10k, Resistor_THT:R_Axial_DIN0207_L6.3mm_D2.5mm_P10.16mm_Horizontal, symbol Device:R
- removed R?: 47k, Resistor_THT:R_Axial_DIN0207_L6.3mm_D2.5mm_P10.16mm_Horizontal, symbol Device:R
- removed U?: NE555, symbol Timer:NE555
- added C12, C13, C14: 1u, Capacitor_THT:CP_Radial_D5.0mm_P2.50mm, symbol Device:CP1
- added D5, D6, D7: 1N4148, Diode_THT:D_DO-35_SOD27_P7.62mm_Horizontal, symbol Device:D
- added J9: ctrl_2, Connector_PinHeader_2.54mm:PinHeader_1x04_P2.54mm_Vertical, symbol Connector_Generic:Conn_01x04
- added Q2, Q3, Q4, Q5: BC546B, Package_TO_SOT_THT:TO-92_Inline_Wide, symbol Device:Q_NPN_CBE
- added Q6, Q7, Q8: BC556B, Package_TO_SOT_THT:TO-92_Inline_Wide, symbol Device:Q_PNP_BCE
- added R10, R12, R14, R15: 100k, Resistor_THT:R_Axial_DIN0207_L6.3mm_D2.5mm_P10.16mm_Horizontal, symbol Device:R
- added R11, R13: 100, Resistor_THT:R_Axial_DIN0207_L6.3mm_D2.5mm_P10.16mm_Horizontal, symbol Device:R
- added R16, R17, R18, R19, R20: 22k, Resistor_THT:R_Axial_DIN0207_L6.3mm_D2.5mm_P10.16mm_Horizontal, symbol Device:R
- added R8: 47k, Resistor_THT:R_Axial_DIN0207_L6.3mm_D2.5mm_P10.16mm_Horizontal, symbol Device:R
- J5: value left_power -> power_1
- J6: value right_power -> power_2
- J7: renamed from J?; value left_power -> signal
- J8: renamed from J?; value left_power -> ctrl_1
- R9: value 47k -> 100k; Manufacturer Vishay: SFR2500001002JA500 -> (none); Manufacturer1 (none) -> Multicomp: MF12 100K; Manufacturer2 (none) -> Yageo: CFR-12JB-52-100K; Supplier1 Farnell:9476539 -> Farnell: 9342427; Supplier2 (none) -> Mouser: 603-CFR-12JB-52-100K; Type MF -> CF
- gave numbers to parts that had none: 2
Connections:
- net labels added: ac_detect, clipping, mute_control
- wire segments 160 -> 229
- no-connect marks 1 -> 2
Other:
- note added: "TDA7293 datasheet specify a test\nwhich uses 0.5mA current. Calculate\nthis resistance as Vcc/0.5mA."
- moved on the sheet: C1, C10, C11, C2, C3, C4, C5, C6, C7, C8, C9, D1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

Commit message: Preliminary placement of AC detect and clipping circuitry.
Signed-off-by: Nenad Radulovic <nenad.b.radulovic@gmail.com>
Parts:
- added C15: 10u, Capacitor_THT:CP_Radial_D8.0mm_P2.50mm, symbol Device:CP1
- C12, C14: value 1u -> 2u2
- C13: value 1u -> 4u7
- J7: footprint Connector_PinHeader_2.54mm:PinHeader_1x04_P2.54mm_Vertical -> Connector_PinHeader_2.54mm:PinHeader_1x03_P2.54mm_Vertical
- Q6, Q7, Q8: symbol Device:Q_PNP_BCE -> Device:Q_PNP_CBE
- R21, R22: value 10k -> 4k7; footprint Resistor_THT:R_Axial_DIN0207_L6.3mm_D2.5mm_P10.16mm_Horizontal -> Resistor_THT:R_Axial_DIN0309_L9.0mm_D3.2mm_P12.70mm_Horizontal; Power 0.4W -> 0.5W
Connections:
- net GNDPWR: now also Q8.1 (C), C15.2; no longer Q8.2 (C)
- net vcc: now also C15.1
- net at Q5.1 (C), R15.2: now also Q7.2 (B); no longer Q7.1 (B)
- net at D7.2 (A), R20.1: now also Q7.1 (C), Q8.2 (B); no longer Q7.2 (C), Q8.1 (B)
- net at J7.1 (Pin_1): now also R22.1; no longer R22.2
- net at Q6.2 (B): now also Q4.1 (C), R14.2; no longer R22.1
- new net: Q6.1 (C), R22.2
Changed lines of the file:
@@
 F 0 "J7" H 10720 2617 50  0000 C CNN
 F 1 "signal" H 10720 2526 50  0000 C CNN
-F 2 "Connector_PinHeader_2.54mm:PinHeader_1x04_P2.54mm_Vertical" H 10800 2300 50  0001 C CNN
+F 2 "Connector_PinHeader_2.54mm:PinHeader_1x03_P2.54mm_Vertical" H 10800 2300 50  0001 C CNN
 F 3 "http://www.farnell.com/datasheets/2138271.pdf" H 10800 2300 50  0001 C CNN
 F 4 "Phoenix: 1803439 (MCV 1,5/ 3-G-3,81)" H 10800 2300 50  0001 C CNN "Manufacturer"
@@
 L power:GNDPWR #PWR08
 U 1 1 5CE10132
-P 9700 6200
-F 0 "#PWR08" H 9700 6000 50  0001 C CNN
-F 1 "GNDPWR" V 9704 6091 50  0000 R CNN
-F 2 "" H 9700 6150 50  0001 C CNN
-F 3 "" H 9700 6150 50  0001 C CNN
-	1    9700 6200
+P 10200 6200
+F 0 "#PWR08" H 10200 6000 50  0001 C CNN
+F 1 "GNDPWR" V 10204 6091 50  0000 R CNN
+F 2 "" H 10200 6150 50  0001 C CNN
+F 3 "" H 10200 6150 50  0001 C CNN
+	1    10200 6200
 	0    -1   -1   0
 $EndComp
@@
 P 9950 2400
 F 0 "R21" V 10065 2400 50  0000 C CNN
-F 1 "10k" V 10156 2400 50  0000 C CNN
-F 2 "Resistor_THT:R_Axial_DIN0207_L6.3mm_D2.5mm_P10.16mm_Horizontal" V 9880 2400 50  0001 C CNN
+F 1 "4k7" V 10156 2400 50  0000 C CNN
+F 2 "Resistor_THT:R_Axial_DIN0309_L9.0mm_D3.2mm_P12.70mm_Horizontal" V 9880 2400 50  0001 C CNN
 F 3 "https://export.farnell.com/c/passive-components/resistors-fixed-value/through-hole-resistors?product-range=sfr125-series" H 9950 2400 50  0001 C CNN
 F 4 "Vishay: SFR2500001002JA500" H 9950 2400 50  0001 C CNN "Manufacturer"
 F 5 "Farnell:9476539" H 9950 2400 50  0001 C CNN "Supplier1"
-F 6 "0.4W" V 10247 2400 50  0000 C CNN "Power"
+F 6 "0.5W" V 10247 2400 50  0000 C CNN "Power"
 F 7 "MF" V 10338 2400 50  0000 C CNN "Type"
 	1    9950 2400
 	0    1    1    0
-$EndComp
-$Comp
-L Device:R R22
-U 1 1 5CE31138
-P 10350 2200
-F 0 "R22" V 10739 2200 50  0000 C CNN
-F 1 "10k" V 10648 2200 50  0000 C CNN
-F 2 "Resistor_THT:R_Axial_DIN0207_L6.3mm_D2.5mm_P10.16mm_Horizontal" V 10280 2200 50  0001 C CNN
-F 3 "https://export.farnell.com/c/passive-components/resistors-fixed-value/through-hole-resistors?product-range=sfr125-series" H 10350 2200 50  0001 C CNN
-F 4 "Vishay: SFR2500001002JA500" H 10350 2200 50  0001 C CNN "Manufacturer"
-F 5 "Farnell:9476539" H 10350 2200 50  0001 C CNN "Supplier1"
-F 6 "0.4W" V 10557 2200 50  0000 C CNN "Power"
-F 7 "MF" V 10466 2200 50  0000 C CNN "Type"
-	1    10350 2200
-	0    -1   -1   0
 $EndComp
 NoConn ~ 10600 4600
@@
 P 6100 5950
 F 0 "C12" H 6215 6041 50  0000 L CNN
-F 1 "1u" H 6215 5950 50  0000 L CNN
+F 1 "2u2" H 6215 5950 50  0000 L CNN
 F 2 "Capacitor_THT:CP_Radial_D5.0mm_P2.50mm" H 6100 5950 50  0001 C CNN
 F 3 "http://www.farnell.com/datasheets/2045874.pdf" H 6100 5950 50  0001 C CNN
@@
 P 7600 5950
 F 0 "C14" H 7715 6041 50  0000 L CNN
-F 1 "1u" H 7715 5950 50  0000 L CNN
+F 1 "2u2" H 7715 5950 50  0000 L CNN
 F 2 "Capacitor_THT:CP_Radial_D5.0mm_P2.50mm" H 7600 5950 50  0001 C CNN
 F 3 "http://www.farnell.com/datasheets/2045874.pdf" H 7600 5950 50  0001 C CNN
@@
 	7100 4600 7100 5000
 $Comp
-L Device:Q_PNP_BCE Q7
+L Device:Q_PNP_CBE Q7
 U 1 1 5CDF6E6A
 P 9000 4200
@@
 Wire Wire Line
 	9600 4700 9500 4700
-$Comp
-L power:GNDPWR #PWR09
-U 1 1 5CE73A93
-P 10100 6300
-F 0 "#PWR09" H 10100 6100 50  0001 C CNN
-F 1 "GNDPWR" V 10104 6191 50  0000 R CNN
-F 2 "" H 10100 6250 50  0001 C CNN
-F 3 "" H 10100 6250 50  0001 C CNN
-	1    10100 6300
-	1    0    0    -1
-$EndComp
-Wire Wire Line
-	10100 6300 10100 5400
+Wire Wire Line
+	10100 6200 10100 5400
 Wire Wire Line
 	10100 4800 10600 4800
@@
 	7600 4700 7600 5800
 $Comp
-L Device:Q_PNP_BCE Q8
+L Device:Q_PNP_CBE Q8
 U 1 1 5CEE7338
 P 9500 5200
@@
 P 7600 2950
 F 0 "C13" H 7715 3041 50  0000 L CNN
-F 1 "1u" H 7715 2950 50  0000 L CNN
+F 1 "4u7" H 7715 2950 50  0000 L CNN
 F 2 "Capacitor_THT:CP_Radial_D5.0mm_P2.50mm" H 7600 2950 50  0001 C CNN
 F 3 "http://www.farnell.com/datasheets/2045874.pdf" H 7600 2950 50  0001 C CNN
@@
 	7100 1600 7100 2000
 $Comp
-L Device:Q_PNP_BCE Q6
+L Device:Q_PNP_CBE Q6
 U 1 1 5CF4BA66
 P 9000 1200
@@
 Connection ~ 6600 2200
 Wire Wire Line
-	9700 6200 9600 6200
+	10200 6200 10100 6200
 Connection ~ 9600 6200
 Wire Wire Line
@@
 Wire Wire Line
 	6100 700  6600 700
+$Comp
+L Device:R R22
+U 1 1 5CE0308D
+P 10350 2200
+F 0 "R22" V 9961 2200 50  0000 C CNN
+F 1 "4k7" V 10052 2200 50  0000 C CNN
+F 2 "Resistor_THT:R_Axial_DIN0309_L9.0mm_D3.2mm_P12.70mm_Horizontal" V 10280 2200 50  0001 C CNN
+F 3 "https://export.farnell.com/c/passive-components/resistors-fixed-value/through-hole-resistors?product-range=sfr125-series" H 10350 2200 50  0001 C CNN
+F 4 "Vishay: SFR2500001002JA500" H 10350 2200 50  0001 C CNN "Manufacturer"
+F 5 "Farnell:9476539" H 10350 2200 50  0001 C CNN "Supplier1"
+F 6 "0.5W" V 10143 2200 50  0000 C CNN "Power"
+F 7 "MF" V 10234 2200 50  0000 C CNN "Type"
+	1    10350 2200
+	0    1    1    0
+$EndComp
+$Comp
+L Device:CP1 C15
+U 1 1 5CE0402B
+P 4100 950
+F 0 "C15" H 4215 1041 50  0000 L CNN
+F 1 "10u" H 4215 950 50  0000 L CNN
+F 2 "Capacitor_THT:CP_Radial_D8.0mm_P2.50mm" H 4100 950 50  0001 C CNN
+F 3 "http://www.farnell.com/datasheets/2045874.pdf" H 4100 950 50  0001 C CNN
+F 4 "Vishay: MAL225630682E3" H 4100 950 50  0001 C CNN "Manufacturer"
+F 5 "Farnell:2474575" H 4100 950 50  0001 C CNN "Supplier1"
+F 6 "35V" H 4215 859 50  0000 L CNN "Voltage"
+	1    4100 950
+	1    0    0    -1
+$EndComp
+$Comp
+L power:GNDPWR #PWR0101
+U 1 1 5CE04114
+P 4100 1200
+F 0 "#PWR0101" H 4100 1000 50  0001 C CNN
+F 1 "GNDPWR" V 4104 1091 50  0000 R CNN
+F 2 "" H 4100 1150 50  0001 C CNN
+F 3 "" H 4100 1150 50  0001 C CNN
+	1    4100 1200
+	1    0    0    -1
+$EndComp
+Wire Wire Line
+	4100 1200 4100 1100
+Wire Wire Line
+	4100 800  4100 700
+Wire Wire Line
+	4100 700  4600 700
+Connection ~ 4600 700
+Connection ~ 10100 6200
+Wire Wire Line
+	10100 6200 9600 6200
 $EndSCHEMATC

Commit message: Updated to new version v1.02.
Signed-off-by: Nenad Radulovic <nenad.b.radulovic@gmail.com>
Parts:
- removed C12: 2u2, Capacitor_THT:CP_Radial_D5.0mm_P2.50mm, symbol Device:CP1
- removed C13: 4u7, Capacitor_THT:CP_Radial_D5.0mm_P2.50mm, symbol Device:CP1
- removed D3, D4, D5, D6, D7: 1N4148, Diode_THT:D_DO-35_SOD27_P7.62mm_Horizontal, symbol Device:D
- removed Q1, Q2, Q3, Q4, Q5: BC546B, Package_TO_SOT_THT:TO-92_Inline_Wide, symbol Device:Q_NPN_CBE
- removed Q6, Q7, Q8: BC556B, Package_TO_SOT_THT:TO-92_Inline_Wide, symbol Device:Q_PNP_CBE
- removed R10, R12, R14, R15, R9: 100k, Resistor_THT:R_Axial_DIN0207_L6.3mm_D2.5mm_P10.16mm_Horizontal, symbol Device:R
- removed R11, R13: 100, Resistor_THT:R_Axial_DIN0207_L6.3mm_D2.5mm_P10.16mm_Horizontal, symbol Device:R
- removed R16, R17, R18, R19, R20: 22k, Resistor_THT:R_Axial_DIN0207_L6.3mm_D2.5mm_P10.16mm_Horizontal, symbol Device:R
- removed R8: 47k, Resistor_THT:R_Axial_DIN0207_L6.3mm_D2.5mm_P10.16mm_Horizontal, symbol Device:R
- added C12, C15: 470n, Capacitor_THT:C_Rect_L7.2mm_W8.5mm_P5.00mm_FKP2_FKP2_MKS2_MKP2, symbol Device:C
- added J11: signal, Connector_PinHeader_2.54mm:PinHeader_1x03_P2.54mm_Vertical, symbol Connector_Generic:Conn_01x03
- added J8: prog, Connector_PinHeader_2.54mm:PinHeader_1x04_P2.54mm_Vertical, symbol Connector_Generic:Conn_01x05
- added U1: L7805, Package_TO_SOT_THT:TO-220-3_Vertical, symbol Regulator_Linear:L7805
- added U2: PIC18F26K20_ISS, Package_DIP:DIP-28_W7.62mm_LongPads, symbol MCU_Microchip_PIC18:PIC18F26K20_ISS
- C14: value 2u2 -> 10u; footprint Capacitor_THT:CP_Radial_D5.0mm_P2.50mm -> Capacitor_THT:CP_Radial_D8.0mm_P2.50mm
- R8: renamed from R21; value 4k7 -> 1k; footprint Resistor_THT:R_Axial_DIN0309_L9.0mm_D3.2mm_P12.70mm_Horizontal -> Resistor_THT:R_Axial_DIN0207_L6.3mm_D2.5mm_P10.16mm_Horizontal
- R9: renamed from R22; value 4k7 -> 1k; footprint Resistor_THT:R_Axial_DIN0309_L9.0mm_D3.2mm_P12.70mm_Horizontal -> Resistor_THT:R_Axial_DIN0207_L6.3mm_D2.5mm_P10.16mm_Horizontal
- renumbered C15 to C13, J9 to J10, J8 to J9
Connections:
- net GNDPWR: now also C12.2, C15.2, J11.1 (Pin_1), J8.3 (Pin_3), U1.2 (GND), U2.19 (Vss), U2.8 (Vss); no longer R7.2
- net ac_detect: now also R6.2, C12.1, U2.21 (AN12/INT0/RB0)
- net acs_p: now also R6.1
- net clipping: now also U2.22 (AN10/INT1/RB1)
- net mute_control: now also U2.23 (AN8/INT2/RB2); no longer R8.2
- net vcc: now also U1.1 (IN)
- net vdd: now reaches R7.1
- net vdd: now also C14.1, C15.1, J8.1 (Pin_1), U1.3 (OUT), U2.20 (Vdd); no longer R6.2
- net at R9.2: now also U2.24 (AN9/RB3)
- new net: R8.2, U2.25 (AN11/RB4)
- new net: J8.2 (Pin_2), R7.2, U2.1 (~MCLR~/RE3)
- new net: J11.2 (Pin_2), U2.17 (TX/RC6)
- new net: J11.3 (Pin_3), U2.18 (RX/RC7)
- new net: J8.4 (Pin_4), U2.27 (PGC/RB6)
- new net: J8.5 (Pin_5), U2.28 (PGD/RB7)
Other:
- moved on the sheet: C13, J10, J7, J9, R6, R8, R9

Commit message: Project update
Signed-off-by: Nenad Radulovic <nenad.b.radulovic@gmail.com>
Parts:
- removed C12, C15: 470n, Capacitor_THT:C_Rect_L7.2mm_W8.5mm_P5.00mm_FKP2_FKP2_MKS2_MKP2, symbol Device:C
- removed J11: signal, Connector_PinHeader_2.54mm:PinHeader_1x03_P2.54mm_Vertical, symbol Connector_Generic:Conn_01x03
- removed J8: prog, Connector_PinHeader_2.54mm:PinHeader_1x04_P2.54mm_Vertical, symbol Connector_Generic:Conn_01x05
- removed U1: L7805, Package_TO_SOT_THT:TO-220-3_Vertical, symbol Regulator_Linear:L7805
- removed U2: PIC18F26K20_ISS, Package_DIP:DIP-28_W7.62mm_LongPads, symbol MCU_Microchip_PIC18:PIC18F26K20_ISS
- added C12: 2u2, Capacitor_THT:CP_Radial_D5.0mm_P2.50mm, symbol Device:CP1
- added C13: 4u7, Capacitor_THT:CP_Radial_D5.0mm_P2.50mm, symbol Device:CP1
- added D3, D4, D5, D6, D7: 1N4148, Diode_THT:D_DO-35_SOD27_P7.62mm_Horizontal, symbol Device:D
- added Q1, Q2, Q3, Q4, Q5: BC546B, Package_TO_SOT_THT:TO-92_Inline_Wide, symbol Device:Q_NPN_CBE
- added Q6, Q7, Q8: BC556B, Package_TO_SOT_THT:TO-92_Inline_Wide, symbol Device:Q_PNP_CBE
- added R10, R12, R14, R15, R9: 100k, Resistor_THT:R_Axial_DIN0207_L6.3mm_D2.5mm_P10.16mm_Horizontal, symbol Device:R
- added R11, R13: 100, Resistor_THT:R_Axial_DIN0207_L6.3mm_D2.5mm_P10.16mm_Horizontal, symbol Device:R
- added R16, R17, R18, R19, R20: 22k, Resistor_THT:R_Axial_DIN0207_L6.3mm_D2.5mm_P10.16mm_Horizontal, symbol Device:R
- added R8: 47k, Resistor_THT:R_Axial_DIN0207_L6.3mm_D2.5mm_P10.16mm_Horizontal, symbol Device:R
- C14: value 10u -> 2u2; footprint Capacitor_THT:CP_Radial_D8.0mm_P2.50mm -> Capacitor_THT:CP_Radial_D5.0mm_P2.50mm
- R21: renamed from R8; value 1k -> 4k7; footprint Resistor_THT:R_Axial_DIN0207_L6.3mm_D2.5mm_P10.16mm_Horizontal -> Resistor_THT:R_Axial_DIN0309_L9.0mm_D3.2mm_P12.70mm_Horizontal
- R22: renamed from R9; value 1k -> 4k7; footprint Resistor_THT:R_Axial_DIN0207_L6.3mm_D2.5mm_P10.16mm_Horizontal -> Resistor_THT:R_Axial_DIN0309_L9.0mm_D3.2mm_P12.70mm_Horizontal
- renumbered C13 to C15, J9 to J8, J10 to J9
Connections:
- net GNDPWR: now also R7.2, C12.2, C13.2, Q1.3 (E), Q2.3 (E), Q3.3 (E), Q8.1 (C), R17.2, R19.2, R20.2
- net ac_detect: now also C12.1, Q1.1 (C), Q3.2 (B), R9.2; no longer R6.2
- net acs_n: now also D4.2 (A)
- net acs_p: now also D3.2 (A); no longer R6.1
- net clipping: now also Q2.2 (B), R8.2
- net mute_control: now also R21.2, D7.1 (K), Q8.3 (E)
- net vcc: now also Q6.3 (E), Q7.3 (E), R10.1, R12.1, R14.1, R15.1, R16.1, R18.1, R8.1, R9.1
- net at R22.2: now also Q6.1 (C)
- net vdd: no longer names the net of R7.1
- net vdd: now also R6.2, Q1.2 (B); no longer C14.1
- new net: D3.1 (K), D4.1 (K), R6.1
- new net: Q3.1 (C), R13.2
- new net: C14.1, Q5.2 (B), R12.2, R13.1
- new net: D7.2 (A), Q7.1 (C), Q8.2 (B), R20.1
- new net: Q5.1 (C), Q7.2 (B), R15.2
- new net: D6.1 (K), R18.2, R19.1
- new net: D6.2 (A), Q5.3 (E)
- new net: Q2.1 (C), R11.2
- new net: C13.1, Q4.2 (B), R10.2, R11.1
- new net: Q4.1 (C), Q6.2 (B), R14.2
- new net: D5.1 (K), R16.2, R17.1
- new net: D5.2 (A), Q4.3 (E)
Other:
- moved on the sheet: C15, J7, J8, J9, R21, R22, R6
